File: main.sch (EAGLE design)
At the start: 14 parts, among them IC1 ATMEGA328P-PU, IC2 LM7805, J1 2,1mm, Q1 16 MHz

Commit message: Minor fixes
Parts:
- removed C1, C2: 22 pF, capacitor-wima:C2.5/2
- added C10, C11: 22 pF, rcl:C-EU025-025X050
- added C7, C8, C9: 0,1 μF, rcl:C-EU050-025X075
- added D1: 1N4004, diode:1N4004
Connections:
- new net N$12: C8.2, IC1.AREF
- new net N$13: D1.A, J1.3
- net +5V: now also C7.2, C9.1, IC1.AVCC
- net GND: now also C10.1, C11.1, C7.1, C8.1, C9.2; no longer C1.2, C2.2
- net N$1: now also C11.2; no longer C2.1
- net N$2: now also C10.2; no longer C1.1
- net VCC: now also D1.C; no longer J1.3
Other:
- moved on the sheet: C3, C4, C5, IC2, J1, Q1, S1, SV2, U$1

Commit message: Opravy
Parts:
- added C1: 22 pF, rcl:C-EU025-025X050
- added L1: EC24-100K, rcl:L-EU0207/12
- added LED1: Red, led:LED5MM
- added LED2: Green, led:LED5MM
- added LED3: Yellow, led:LED5MM
- added R1, R4, R5, R6, R7, R8: (no value), rcl:R-EU_0207/7
- added R2, R3: 10K, rcl:R-EU_0207/7
- C11: value 22 pF -> 0,1 μF; device rcl:C-EU025-025X050 -> rcl:C-EU050-025X075
- S1: value (none) -> TC-0103-T
- renumbered C10 to C2
Connections:
- new net N$14: IC1.(PCI4/MISO)PB4, R4.1
- new net N$16: IC1.(PCI5/SCK)PB5, R5.1
- new net N$17: LED3.A, R4.2
- new net N$18: C9.1, IC1.AVCC, L1.2
- new net N$19: LED2.A, R5.2
- new net N$20: LED1.A, R6.1
- new net N$21: R8.1, SV1.2
- new net N$22: R7.1, SV1.3
- net +5V: now also L1.1, R1.2, R2.2, R3.2, R6.2; no longer C9.1, IC1.AVCC
- net GND: now also C1.1, C11.2, LED1.C, LED2.C, LED3.C; no longer C11.1
- net N$1: now also C1.2; no longer C11.2
- net N$3: now also R3.1
- net N$4: now also R2.1
- net N$5: now also C6.1, R1.1; no longer C6.2
- net N$6: now also C11.1
- net N$7: now also C6.2; no longer C6.1
- net N$8: now also R7.2; no longer SV1.3
- net N$9: now also R8.2; no longer SV1.2
Other:
- moved on the sheet: C11, C6

Commit message: Revize 0.0.1
Parts:
- R1: value (none) -> 10K
- R4, R5, R6: value (none) -> 330
- R7, R8: value (none) -> 1K
Changed lines of the file:
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@@
 <grid distance="0.1" unitdist="inch" unit="inch" style="lines" multiple="1" display="no" altdistance="0.01" altunitdist="inch" altunit="inch"/>
 <layers>
-<layer number="1" name="Top" color="4" fill="1" visible="yes" active="no"/>
-<layer number="16" name="Bottom" color="1" fill="1" visible="yes" active="no"/>
-<layer number="17" name="Pads" color="2" fill="1" visible="yes" active="no"/>
-<layer number="18" name="Vias" color="2" fill="1" visible="yes" active="no"/>
-<layer number="19" name="Unrouted" color="6" fill="1" visible="yes" active="no"/>
-<layer number="20" name="Dimension" color="15" fill="1" visible="yes" active="no"/>
-<layer number="21" name="tPlace" color="7" fill="1" visible="yes" active="no"/>
-<layer number="22" name="bPlace" color="7" fill="1" visible="yes" active="no"/>
-<layer number="23" name="tOrigins" color="15" fill="1" visible="yes" active="no"/>
-<layer number="24" name="bOrigins" color="15" fill="1" visible="yes" active="no"/>
-<layer number="25" name="tNames" color="7" fill="1" visible="yes" active="no"/>
-<layer number="26" name="bNames" color="7" fill="1" visible="yes" active="no"/>
-<layer number="27" name="tValues" color="7" fill="1" visible="yes" active="no"/>
-<layer number="28" name="bValues" color="7" fill="1" visible="yes" active="no"/>
+<layer number="1" name="Top" color="4" fill="1" visible="no" active="no"/>
+<layer number="16" name="Bottom" color="1" fill="1" visible="no" active="no"/>
+<layer number="17" name="Pads" color="2" fill="1" visible="no" active="no"/>
+<layer number="18" name="Vias" color="2" fill="1" visible="no" active="no"/>
+<layer number="19" name="Unrouted" color="6" fill="1" visible="no" active="no"/>
+<layer number="20" name="Dimension" color="15" fill="1" visible="no" active="no"/>
+<layer number="21" name="tPlace" color="7" fill="1" visible="no" active="no"/>
+<layer number="22" name="bPlace" color="7" fill="1" visible="no" active="no"/>
+<layer number="23" name="tOrigins" color="15" fill="1" visible="no" active="no"/>
+<layer number="24" name="bOrigins" color="15" fill="1" visible="no" active="no"/>
+<layer number="25" name="tNames" color="7" fill="1" visible="no" active="no"/>
+<layer number="26" name="bNames" color="7" fill="1" visible="no" active="no"/>
+<layer number="27" name="tValues" color="7" fill="1" visible="no" active="no"/>
+<layer number="28" name="bValues" color="7" fill="1" visible="no" active="no"/>
 <layer number="29" name="tStop" color="7" fill="3" visible="no" active="no"/>
 <layer number="30" name="bStop" color="7" fill="6" visible="no" active="no"/>
@@
 <layer number="35" name="tGlue" color="7" fill="4" visible="no" active="no"/>
 <layer number="36" name="bGlue" color="7" fill="5" visible="no" active="no"/>
-<layer number="37" name="tTest" color="7" fill="1" visible="yes" active="no"/>
-<layer number="38" name="bTest" color="7" fill="1" visible="yes" active="no"/>
+<layer number="37" name="tTest" color="7" fill="1" visible="no" active="no"/>
+<layer number="38" name="bTest" color="7" fill="1" visible="no" active="no"/>
 <layer number="39" name="tKeepout" color="4" fill="11" visible="no" active="no"/>
 <layer number="40" name="bKeepout" color="1" fill="11" visible="no" active="no"/>
@@
 <layer number="44" name="Drills" color="7" fill="1" visible="no" active="no"/>
 <layer number="45" name="Holes" color="7" fill="1" visible="no" active="no"/>
-<layer number="46" name="Milling" color="3" fill="1" visible="yes" active="no"/>
-<layer number="47" name="Measures" color="7" fill="1" visible="yes" active="no"/>
-<layer number="48" name="Document" color="7" fill="1" visible="yes" active="no"/>
-<layer number="49" name="Reference" color="7" fill="1" visible="yes" active="no"/>
-<layer number="50" name="dxf" color="7" fill="1" visible="yes" active="no"/>
-<layer number="51" name="tDocu" color="7" fill="1" visible="yes" active="no"/>
-<layer number="52" name="bDocu" color="7" fill="1" visible="yes" active="no"/>
-<layer number="53" name="tGND_GNDA" color="7" fill="9" visible="yes" active="no"/>
-<layer number="54" name="bGND_GNDA" color="1" fill="9" visible="yes" active="no"/>
-<layer number="56" name="wert" color="7" fill="1" visible="yes" active="no"/>
-<layer number="57" name="tCAD" color="7" fill="1" visible="yes" active="no"/>
+<layer number="46" name="Milling" color="3" fill="1" visible="no" active="no"/>
+<layer number="47" name="Measures" color="7" fill="1" visible="no" active="no"/>
+<layer number="48" name="Document" color="7" fill="1" visible="no" active="no"/>
+<layer number="49" name="Reference" color="7" fill="1" visible="no" active="no"/>
+<layer number="50" name="dxf" color="7" fill="1" visible="no" active="no"/>
+<layer number="51" name="tDocu" color="7" fill="1" visible="no" active="no"/>
+<layer number="52" name="bDocu" color="7" fill="1" visible="no" active="no"/>
+<layer number="53" name="tGND_GNDA" color="7" fill="9" visible="no" active="no"/>
+<layer number="54" name="bGND_GNDA" color="1" fill="9" visible="no" active="no"/>
+<layer number="56" name="wert" color="7" fill="1" visible="no" active="no"/>
+<layer number="57" name="tCAD" color="7" fill="1" visible="no" active="no"/>
 <layer number="90" name="Modules" color="5" fill="1" visible="yes" active="yes"/>
 <layer number="91" name="Nets" color="2" fill="1" visible="yes" active="yes"/>
@@
 <part name="C1" library="rcl" library_urn="urn:adsk.eagle:library:334" deviceset="C-EU" device="025-025X050" value="22 pF"/>
 <part name="L1" library="rcl" library_urn="urn:adsk.eagle:library:334" deviceset="L-EU" device="0207/12" value="EC24-100K"/>
-<part name="R1" library="rcl" library_urn="urn:adsk.eagle:library:334" deviceset="R-EU_" device="0207/7"/>
+<part name="R1" library="rcl" library_urn="urn:adsk.eagle:library:334" deviceset="R-EU_" device="0207/7" value="10K"/>
 <part name="P+8" library="supply1" library_urn="urn:adsk.eagle:library:371" deviceset="+5V" device=""/>
 <part name="R2" library="rcl" library_urn="urn:adsk.eagle:library:334" deviceset="R-EU_" device="0207/7" value="10K"/>
@@
 <part name="LED2" library="led" library_urn="urn:adsk.eagle:library:259" deviceset="LED" device="5MM" value="Green"/>
 <part name="LED3" library="led" library_urn="urn:adsk.eagle:library:259" deviceset="LED" device="5MM" value="Yellow"/>
-<part name="R4" library="rcl" library_urn="urn:adsk.eagle:library:334" deviceset="R-EU_" device="0207/7"/>
-<part name="R5" library="rcl" library_urn="urn:adsk.eagle:library:334" deviceset="R-EU_" device="0207/7"/>
+<part name="R4" library="rcl" library_urn="urn:adsk.eagle:library:334" deviceset="R-EU_" device="0207/7" value="330"/>
+<part name="R5" library="rcl" library_urn="urn:adsk.eagle:library:334" deviceset="R-EU_" device="0207/7" value="330"/>
 <part name="GND12" library="supply1" library_urn="urn:adsk.eagle:library:371" deviceset="GND" device=""/>
-<part name="R6" library="rcl" library_urn="urn:adsk.eagle:library:334" deviceset="R-EU_" device="0207/7"/>
+<part name="R6" library="rcl" library_urn="urn:adsk.eagle:library:334" deviceset="R-EU_" device="0207/7" value="330"/>
 <part name="P+11" library="supply1" library_urn="urn:adsk.eagle:library:371" deviceset="+5V" device=""/>
 <part name="GND13" library="supply1" library_urn="urn:adsk.eagle:library:371" deviceset="GND" device=""/>
-<part name="R7" library="rcl" library_urn="urn:adsk.eagle:library:334" deviceset="R-EU_" device="0207/7"/>
-<part name="R8" library="rcl" library_urn="urn:adsk.eagle:library:334" deviceset="R-EU_" device="0207/7"/>
+<part name="R7" library="rcl" library_urn="urn:adsk.eagle:library:334" deviceset="R-EU_" device="0207/7" value="1K"/>
+<part name="R8" library="rcl" library_urn="urn:adsk.eagle:library:334" deviceset="R-EU_" device="0207/7" value="1K"/>
 </parts>
 <sheets>

Commit message: Opravy na celorepublikové kolo
Parts:
- OLED: value OLED_0.96_I2C -> 128x64 SSD1306 I2C
- renumbered U$1 to OLED
Connections:
- net N$13 renamed IJVCC
- net N$4 renamed SCL
- net N$6 renamed BTN
Other:
- moved on the sheet: R5, R8
Changed lines of the file:
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@@
 <?xml version="1.0" encoding="utf-8"?>
 <!DOCTYPE eagle SYSTEM "eagle.dtd">
-<eagle version="8.2.0">
+<eagle version="8.2.1">
 <drawing>
 <settings>
@@
 <part name="C6" library="rcl" library_urn="urn:adsk.eagle:library:334" deviceset="C-EU" device="050-025X075" value="0,1 μF"/>
 <part name="P+6" library="supply1" library_urn="urn:adsk.eagle:library:371" deviceset="VCC" device=""/>
-<part name="U$1" library="tft_1.8_1.44_oled_0.96" deviceset="OLED_0.96_I2C" device=""/>
+<part name="OLED" library="tft_1.8_1.44_oled_0.96" deviceset="OLED_0.96_I2C" device="" value="128x64 SSD1306 I2C"/>
 <part name="IC2" library="78xx_with_heatsink" deviceset="78XXH" device="" value="LM7805"/>
 <part name="GND7" library="supply1" library_urn="urn:adsk.eagle:library:371" deviceset="GND" device=""/>
@@
 <instance part="C6" gate="G$1" x="73.66" y="104.14" rot="R90"/>
 <instance part="P+6" gate="VCC" x="187.96" y="119.38"/>
-<instance part="U$1" gate="G$1" x="198.12" y="60.96" rot="R270"/>
+<instance part="OLED" gate="G$1" x="198.12" y="60.96" rot="R270"/>
 <instance part="IC2" gate="A" x="101.6" y="124.46"/>
 <instance part="GND7" gate="1" x="83.82" y="88.9" rot="R180"/>
@@
 <instance part="LED3" gate="G$1" x="152.4" y="33.02" rot="R90"/>
 <instance part="R4" gate="G$1" x="144.78" y="33.02"/>
-<instance part="R5" gate="G$1" x="144.78" y="27.94"/>
+<instance part="R5" gate="G$1" x="144.78" y="25.4"/>
 <instance part="GND12" gate="1" x="160.02" y="27.94" rot="R90"/>
 <instance part="R6" gate="G$1" x="175.26" y="93.98" rot="R90"/>
@@
 <instance part="GND13" gate="1" x="175.26" y="78.74"/>
 <instance part="R7" gate="G$1" x="157.48" y="99.06"/>
-<instance part="R8" gate="G$1" x="152.4" y="96.52"/>
+<instance part="R8" gate="G$1" x="147.32" y="96.52"/>
 </instances>
 <busses>
@@
 <pinref part="GND5" gate="1" pin="GND"/>
 <wire x1="187.96" y1="63.5" x2="177.8" y2="63.5" width="0.1524" layer="91"/>
-<pinref part="U$1" gate="G$1" pin="GND"/>
+<pinref part="OLED" gate="G$1" pin="GND"/>
 </segment>
 <segment>
@@
 <wire x1="187.96" y1="66.04" x2="185.42" y2="66.04" width="0.1524" layer="91"/>
 <wire x1="185.42" y1="66.04" x2="185.42" y2="68.58" width="0.1524" layer="91"/>
-<pinref part="U$1" gate="G$1" pin="VCC"/>
+<pinref part="OLED" gate="G$1" pin="VCC"/>
 </segment>
 <segment>
@@
 <wire x1="167.64" y1="73.66" x2="167.64" y2="58.42" width="0.1524" layer="91"/>
 <wire x1="167.64" y1="58.42" x2="180.34" y2="58.42" width="0.1524" layer="91"/>
-<pinref part="U$1" gate="G$1" pin="SDA"/>
+<pinref part="OLED" gate="G$1" pin="SDA"/>
 <wire x1="180.34" y1="58.42" x2="187.96" y2="58.42" width="0.1524" layer="91"/>
 <wire x1="144.78" y1="81.28" x2="144.78" y2="73.66" width="0.1524" layer="91"/>
@@
 </segment>
 </net>
-<net name="N$4" class="0">
+<net name="SCL" class="0">
 <segment>
 <pinref part="IC1" gate="G$1" pin="(PCI13/ADC5/SCL)PC5"/>
@@
 <wire x1="142.24" y1="78.74" x2="142.24" y2="71.12" width="0.1524" layer="91"/>
 <wire x1="142.24" y1="71.12" x2="170.18" y2="71.12" width="0.1524" layer="91"/>
-<pinref part="U$1" gate="G$1" pin="SCL"/>
+<pinref part="OLED" gate="G$1" pin="SCL"/>
 <wire x1="170.18" y1="60.96" x2="172.72" y2="60.96" width="0.1524" layer="91"/>
 <pinref part="R2" gate="G$1" pin="1"/>
@@
 <wire x1="162.56" y1="63.5" x2="139.7" y2="63.5" width="0.1524" layer="91"/>
 <pinref part="R8" gate="G$1" pin="2"/>
-<wire x1="162.56" y1="96.52" x2="157.48" y2="96.52" width="0.1524" layer="91"/>
-</segment>
-</net>
-<net name="N$6" class="0">
+<wire x1="162.56" y1="96.52" x2="152.4" y2="96.52" width="0.1524" layer="91"/>
+</segment>
+</net>
+<net name="BTN" class="0">
 <segment>
 <pinref part="IC1" gate="G$1" pin="(PCI23/AIN1)PD7"/>
@@
 </segment>
 </net>
-<net name="N$13" class="0">
+<net name="IJVCC" class="0">
 <segment>
 <pinref part="J1" gate="G$1" pin="3"/>
@@
 <pinref part="IC1" gate="G$1" pin="(PCI5/SCK)PB5"/>
 <pinref part="R5" gate="G$1" pin="1"/>
-<wire x1="139.7" y1="27.94" x2="139.7" y2="30.48" width="0.1524" layer="91"/>
+<wire x1="139.7" y1="25.4" x2="139.7" y2="30.48" width="0.1524" layer="91"/>
 </segment>
 </net>
@@
 <pinref part="R5" gate="G$1" pin="2"/>
 <pinref part="LED2" gate="G$1" pin="A"/>
-<wire x1="149.86" y1="22.86" x2="149.86" y2="27.94" width="0.1524" layer="91"/>
+<wire x1="149.86" y1="22.86" x2="149.86" y2="25.4" width="0.1524" layer="91"/>
 </segment>
 </net>
@@
 <wire x1="139.7" y1="111.76" x2="139.7" y2="96.52" width="0.1524" layer="91"/>
 <pinref part="R8" gate="G$1" pin="1"/>
-<wire x1="147.32" y1="96.52" x2="139.7" y2="96.52" width="0.1524" layer="91"/>
+<wire x1="142.24" y1="96.52" x2="139.7" y2="96.52" width="0.1524" layer="91"/>
 </segment>
 </net>
@@
 </sheet>
 </sheets>
+<errors>
+</errors>
 </schematic>
 </drawing>
